Commit message: [ackermann] Add first test with wrong config

File: ackermann_controller/test/urdf/wheel.xacro (robot description, xacro)
@@ -1,40 +1,62 @@
 <?xml version="1.0"?>
-<robot xmlns:xacro="http://www.ros.org/wiki/xacro">
-  <xacro:macro name="wheel" params="name parent radius thickness *origin">
-    <link name="${name}_link">
-      <inertial>
-        <origin xyz="0 0 0" rpy="0 0 0"/>
-        <mass value="1"/>
-        <inertia ixx="0.2" ixy="0" ixz="0" iyy="0.2" iyz="0" izz="0.2"/>
+<robot xmlns:xacro="http://www.ros.org/wiki/xacro" name="wheel">
+  <!--<xacro:property name="M_PI" default="3.14159"/>-->
+  <!-- Wheel Properties -->
+  <xacro:property name="wheel_length" value="0.1" />
+  <xacro:property name="wheel_radius" value="0.28" />
+  <xacro:property name="mass_wheel" value="5.0" />
+  <xacro:macro name="wheel" params="wheel_prefix parent_link left_right *joint_origin">
+    <gazebo reference="${wheel_prefix}_wheel_link">
+      <material>Gazebo/Black</material>
+    </gazebo>
+		<link name="${wheel_prefix}_wheel_link">
+			<inertial>
+        <mass value="${mass_wheel}" />
+        <origin xyz="0 0 0" rpy="${M_PI/2}  0 0" />
+        <!--<inertia ixx="1.0" ixy="0" ixz="0"
+                 iyy="1.0" iyz="0"
+                 izz="1.0"/>-->
+        <inertia  ixx="${mass_wheel/4.0*(wheel_radius*wheel_radius+wheel_length*wheel_length/3.0)}" ixy="0" ixz="0"
+                  iyy="${mass_wheel*wheel_radius*wheel_radius/2.0}" iyz="0"
+                  izz="${mass_wheel/4.0*(wheel_radius*wheel_radius+wheel_length*wheel_length/3.0)}" />
       </inertial>
-      <visual>
-        <origin xyz="0 0 0" rpy="0 0 0"/>
-        <geometry>
-          <cylinder radius="${radius}" length="${thickness}"/>
-        </geometry>
-      </visual>
-      <collision>
-        <origin xyz="0 0 0" rpy="0 0 0"/>
-        <geometry>
-          <cylinder radius="${radius}" length="${thickness}"/>
-        </geometry>
-      </collision>
-    </link>
-    <joint name="${name}_joint" type="continuous">
-      <parent link="${parent}_link"/>
-      <child link="${name}_link"/>
-      <xacro:insert_block name="origin"/>
-      <axis xyz="0 0 1"/>
-    </joint>
-    <!-- Transmission is important to link the joints and the controller -->
-    <transmission name="${name}_joint_trans" type="SimpleTransmission">
-      <actuator name="${name}_joint_motor"/>
-      <joint name="${name}_joint"/>
-      <mechanicalReduction>1</mechanicalReduction>
-      <motorTorqueConstant>1</motorTorqueConstant>
-    </transmission>
-    <gazebo reference="${name}_link">
-      <material>Gazebo/Red</material>
-    </gazebo>
-  </xacro:macro>
+			<visual>
+        <origin xyz="0 0 0" rpy="${left_right * M_PI/2}  0 0" />
+				<geometry>
+          <cylinder length="${wheel_length}" radius="${wheel_radius}"/>
+				</geometry>
+        <material name="black">
+          <color rgba="0 0 0 1"/>
+        </material>
+			</visual>
+			<collision>
+				<origin xyz="0 0 0" rpy="${M_PI/2} 0 0" />
+				<geometry>
+					<cylinder length="${wheel_length}" radius="${wheel_radius}" />
+				</geometry>
+			</collision>
+		</link>
+		<gazebo reference="${wheel_prefix}_wheel_link">
+			<mu1 value="1.0"/>
+			<mu2 value="1.0"/>
+			<kp value="10000000.0" />
+			<kd value="1.0" />
+			<fdir1 value="1 0 0"/>
+		</gazebo>
+		<joint name="${wheel_prefix}_wheel" type="continuous">
+      <parent link="${parent_link}"/>
+			<child link="${wheel_prefix}_wheel_link"/>
+      <xacro:insert_block name="joint_origin"/>
+			<axis xyz="0 1 0" rpy="0 0 0" />
+		</joint>
+		<transmission name="${wheel_prefix}_wheel_trans" type="SimpleTransmission">
+			<type>transmission_interface/SimpleTransmission</type>
+			<actuator name="${wheel_prefix}_wheel_motor">
+				<mechanicalReduction>1</mechanicalReduction>
+			</actuator>
+			<joint name="${wheel_prefix}_wheel">
+				<hardwareInterface>VelocityJointInterface</hardwareInterface>
+			</joint>
+		</transmission>
+	</xacro:macro>
 </robot>

File: ackermann_controller/test/urdf/wheel_steered.xacro (robot description, xacro)
@@ -3,7 +3,7 @@
   <xacro:property name="steering_link_y" value="0.05" />
   <xacro:property name="steering_link_xz" value="0.1" />
-  <xacro:property name="steering_link_mass" value="30.0" />
+  <xacro:property name="steering_link_mass" value="5.0" />
   <xacro:include filename="$(find ackermann_controller)/test/urdf/wheel.xacro" />
-  <xacro:macro name="wheel_steered" params="wheel_prefix parent_link wheel_origin_y *joint_origin ">
+  <xacro:macro name="wheel_steered" params="wheel_prefix parent_link wheel_origin_y left_right *joint_origin ">
     <link name="${wheel_prefix}_steering">
       <visual>
@@ -19,7 +19,10 @@
         <mass value="${steering_link_mass}" />
         <origin xyz="0 ${-wheel_origin_y} 0" />
-        <inertia ixx="0.8" ixy="0" ixz="0"
-                 iyy="0.4" iyz="0"
-                 izz="0.8"/>
+        <!--<inertia ixx="1.0" ixy="0" ixz="0"
+                 iyy="1.0" iyz="0"
+                 izz="1.0"/>-->
+        <inertia  ixx="${steering_link_mass/12.0 * (steering_link_y*steering_link_y + steering_link_xz*steering_link_xz)}" ixy="0" ixz="0"
+                  iyy="${steering_link_mass/12.0 * (steering_link_xz*steering_link_xz + steering_link_xz*steering_link_xz)}" iyz="0"
+                  izz="${steering_link_mass/12.0 * (steering_link_y*steering_link_y + steering_link_xz*steering_link_xz)}" />
       </inertial>
     </link>
@@ -30,8 +33,10 @@
       <child link="${wheel_prefix}_steering"/>
       <xacro:insert_block name="joint_origin"/>
+      <dynamics damping="0.7"/>
     </joint>
     <transmission name="${wheel_prefix}_steering_trans" type="SimpleTransmission">
       <type>transmission_interface/SimpleTransmission</type>
       <actuator name="${wheel_prefix}_steering_motor">
+        <hardwareInterface>PositionJointInterface</hardwareInterface>
         <mechanicalReduction>1</mechanicalReduction>
       </actuator>
@@ -40,5 +45,5 @@
       </joint>
     </transmission>
-    <xacro:wheel wheel_prefix="${wheel_prefix}" parent_link="${wheel_prefix}_steering">
+    <xacro:wheel wheel_prefix="${wheel_prefix}" parent_link="${wheel_prefix}_steering" left_right="${left_right}">
       <origin xyz="0 ${wheel_origin_y} 0" rpy="0 0 0" />
     </xacro:wheel>
